File: ESP32_Dev_Board/ESP32_Dev_Board.kicad_pcb (KiCad board)
At the start: 2 copper layers, 47.2 x 29 mm, 20 parts, among them J1 USB_C_Receptacle_USB2.0_16P, J2 Conn_01x18, J3 Conn_01x18, SW1 SW_RESET, SW2 SW_BOOT, U1 LD1117S33TR_SOT223, U2 ESP32-S3-WROOM-1

Commit message: v0.2 - AP2114 3.3V regulator; Updated capacitor component selection and footprints
Parts:
- C1: value 0.1uF -> 10uF; footprint Capacitor_SMD:C_0603_1608Metric -> Capacitor_SMD:C_0805_2012Metric
- C3: value 10uF -> 22uF; footprint Capacitor_SMD:C_0603_1608Metric -> Capacitor_SMD:C_0805_2012Metric
- C6: footprint Capacitor_SMD:C_0603_1608Metric -> Capacitor_SMD:C_0805_2012Metric
- U1: value LD1117S33TR_SOT223 -> AP2114H-3.3
- moved C1 0.33 mm to (143.2, 105.8)
- moved C5 0.24 mm to (149.0, 95.4)
- moved C2 0.10 mm to (137.8, 92.2)
- moved C3 0.10 mm to (151.3, 102.0)
- moved SW1 0.10 mm to (133.0, 93.8)
- moved SW2 0.10 mm to (132.9, 109.4)
