File: ESP32_Dev_Board/ESP32_Dev_Board.kicad_sch (KiCad schematic)
At the start: 0 parts

Commit message: Version 0.1 - Copleted schematic and PCB design for v0.1, including modified component footprints
Parts:
- added C1, C2, C5: 0.1uF, Capacitor_SMD:C_0603_1608Metric, symbol Device:C
- added C3: 10uF, Capacitor_SMD:C_0603_1608Metric, symbol Device:C
- added C4: 1uF, Capacitor_SMD:C_0603_1608Metric, symbol Device:C
- added C6: 22uF, Capacitor_SMD:C_0603_1608Metric, symbol Device:C
- added D1, D2: LED, Diode_SMD:D_0603_1608Metric, symbol Device:LED
- added J1: USB_C_Receptacle_USB2.0_16P, ESP32_Dev_Board:USB_C_Receptacle_GCT_USB4105-xx-A_16P_TopMnt_Horizontal, symbol Connector:USB_C_Receptacle_USB2.0_16P
- added J2, J3: Conn_01x18, Connector_PinHeader_2.54mm:PinHeader_1x18_P2.54mm_Vertical, symbol Connector_Generic:Conn_01x18
- added R1, R2, R3, R4: 5.1k, Resistor_SMD:R_0603_1608Metric, symbol Device:R
- added R5: 10k, Resistor_SMD:R_0603_1608Metric, symbol Device:R
- added SW1: SW_RESET, Button_Switch_SMD:SW_SPST_TS-1088-xR020, symbol Switch:SW_Push
- added SW2: SW_BOOT, Button_Switch_SMD:SW_SPST_TS-1088-xR020, symbol Switch:SW_Push
- added U1: LD1117S33TR_SOT223, Package_TO_SOT_SMD:SOT-223-3_TabPin2, symbol Regulator_Linear:LD1117S33TR_SOT223
- added U2: ESP32-S3-WROOM-1, ESP32_Dev_Board:ESP32-S3-WROOM-1, symbol RF_Module:ESP32-S3-WROOM-1
Connections:
- new net: J1.B5 (CC2), R3.1
- new net: D1.2 (A), R1.2
- new net: D2.2 (A), R2.2
- new net: J1.A5 (CC1), R4.2
- new net +3V3: C3.1, C5.1, C6.1, J2.1 (Pin_1), R1.1, R5.1, U1.2 (VO), U2.2 (3V3)
- new net +VBUS: C1.1, J1.A4 (VBUS), J1.A9 (VBUS), J1.B4 (VBUS), J1.B9 (VBUS), J3.18 (Pin_18), U1.3 (VI)
- new net D+: J1.A6 (D+), J1.B6 (D+), U2.14 (USB_D+)
- new net D-: J1.A7 (D-), J1.B7 (D-), U2.13 (USB_D-)
- new net GND: C1.2, C2.2, C3.2, C4.2, C5.2, C6.2, D1.1 (K), D2.1 (K), J1.A1 (GND), J1.A12 (GND), J1.B1 (GND), J1.B12 (GND), J1.S1 (SHIELD), J2.2 (Pin_2), J3.1 (Pin_1), R3.2, R4.1, SW1.1, SW2.1, U1.1 (GND), U2.1 (GND), U2.40 (GND), U2.41 (GND)
- new net IO0: J3.11 (Pin_11), SW2.2, U2.27 (IO0)
- new net IO1: J3.2 (Pin_2), U2.39 (IO1)
- new net IO10: J2.16 (Pin_16), U2.18 (IO10)
- new net IO11: J2.17 (Pin_17), U2.19 (IO11)
- new net IO12: J2.18 (Pin_18), U2.20 (IO12)
- new net IO13: J3.17 (Pin_17), U2.21 (IO13)
- new net IO14: J3.16 (Pin_16), U2.22 (IO14)
- new net IO15: J2.8 (Pin_8), U2.8 (IO15)
- new net IO16: J2.9 (Pin_9), U2.9 (IO16)
- new net IO17: J2.10 (Pin_10), U2.10 (IO17)
- new net IO18: J2.11 (Pin_11), U2.11 (IO18)
- new net IO2: J3.3 (Pin_3), U2.38 (IO2)
- new net IO21: J3.15 (Pin_15), R2.1, U2.23 (IO21)
- new net IO3: J2.13 (Pin_13), U2.15 (IO3)
- new net IO38: J3.10 (Pin_10), U2.31 (IO38)
- new net IO39: J3.9 (Pin_9), U2.32 (IO39)
- new net IO4: J2.4 (Pin_4), U2.4 (IO4)
- new net IO40: J3.8 (Pin_8), U2.33 (IO40)
- new net IO41: J3.7 (Pin_7), U2.34 (IO41)
- new net IO42: J3.6 (Pin_6), U2.35 (IO42)
- new net IO43: J3.4 (Pin_4), U2.37 (TXD0)
- new net IO44: J3.5 (Pin_5), U2.36 (RXD0)
- new net IO45: J3.12 (Pin_12), U2.26 (IO45)
- new net IO46: J2.14 (Pin_14), U2.16 (IO46)
- new net IO47: J3.14 (Pin_14), U2.24 (IO47)
- new net IO48: J3.13 (Pin_13), U2.25 (IO48)
- new net IO5: J2.5 (Pin_5), U2.5 (IO5)
- new net IO6: J2.6 (Pin_6), U2.6 (IO6)
- new net IO7: J2.7 (Pin_7), U2.7 (IO7)
- new net IO8: J2.12 (Pin_12), U2.12 (IO8)
- new net IO9: J2.15 (Pin_15), U2.17 (IO9)
- new net RESET: C2.1, C4.1, J2.3 (Pin_3), R5.2, SW1.2, U2.3 (EN)
- no-connect marks 0 -> 5
Other:
- note added: "ESP32-S3-WROOM-1"
- note added: "Header Pins"
- note added: "LEDs"
- note added: "RESET/BOOT Buttons"
- note added: "USB-C"
- note added: "Voltage Regulator"
- title: (none) -> ESP32-S3-WROOM-1 Development Board

Commit message: Update readme
Parts:
- added U3: USBLC6-2SC6, Package_TO_SOT_SMD:SOT-23-6, symbol Power_Protection:USBLC6-2SC6
Other:
- moved on the sheet: C1, C2, C3, C4, C5, C6, J2, J3, R5, SW1, SW2, U1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

Commit message: v0.2 - AP2114 3.3V regulator; Updated capacitor component selection and footprints
Parts:
- removed U3: USBLC6-2SC6, Package_TO_SOT_SMD:SOT-23-6, symbol Power_Protection:USBLC6-2SC6
- C1: value 0.1uF -> 10uF; footprint Capacitor_SMD:C_0603_1608Metric -> Capacitor_SMD:C_0805_2012Metric; LCSC C14663 -> C15850
- C3: value 10uF -> 22uF; footprint Capacitor_SMD:C_0603_1608Metric -> Capacitor_SMD:C_0805_2012Metric; LCSC C19702 -> C45783
- C4: LCSC C15849 -> C15849
- C6: footprint Capacitor_SMD:C_0603_1608Metric -> Capacitor_SMD:C_0805_2012Metric; LCSC C59461 -> C45783
- U1: value LD1117S33TR_SOT223 -> AP2114H-3.3; symbol Regulator_Linear:LD1117S33TR_SOT223 -> ESP32_Dev_Board:AP2114H-3.3; LCSC C86781 -> C150716
Changed lines of the file:
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@@
 	(title_block
 		(title "ESP32-S3-WROOM-1 Development Board")
-		(date "2026-01-14")
-		(rev "v0.1")
+		(date "2026-01-24")
+		(rev "v0.2")
 	)
 	(rectangle
@@
 	)
 	(symbol
-		(lib_id "Power_Protection:USBLC6-2SC6")
-		(at 73.66 48.26 0)
-		(unit 1)
-		(exclude_from_sim no)
-		(in_bom yes)
-		(on_board yes)
-		(dnp no)
-		(fields_autoplaced yes)
-		(property "Reference" "U3"
-			(at 75.3111 40.64 0)
-			(effects
-				(font
-					(size 1.27 1.27)
-				)
-				(justify left)
-			)
-		)
-		(property "Value" "USBLC6-2SC6"
-			(at 75.3111 43.18 0)
-			(effects
-				(font
-					(size 1.27 1.27)
-				)
-				(justify left)
-			)
-		)
-		(property "Footprint" "Package_TO_SOT_SMD:SOT-23-6"
-			(at 74.93 54.61 0)
-			(effects
-				(font
-					(size 1.27 1.27)
-					(italic yes)
-				)
-				(justify left)
-				(hide yes)
-			)
-		)
-		(property "Datasheet" "https://www.st.com/resource/en/datasheet/usblc6-2.pdf"
-			(at 74.93 56.515 0)
-			(effects
-				(font
-					(size 1.27 1.27)
-				)
-				(justify left)
-				(hide yes)
-			)
-		)
-		(property "Description" "Very low capacitance ESD protection diode, 2 data-line, SOT-23-6"
-			(at 73.66 48.26 0)
-			(effects
-				(font
-					(size 1.27 1.27)
-				)
-				(hide yes)
-			)
-		)
-		(property "LCSC" "C7519"
-			(at 73.66 48.26 0)
-			(effects
-				(font
-					(size 1.27 1.27)
-				)
-				(hide yes)
-			)
-		)
-		(pin "1"
-		)
-		(pin "3"
-		)
-		(pin "5"
-		)
-		(pin "2"
-		)
-		(pin "6"
-		)
-		(pin "4"
-		)
-		(instances
-			(project ""
-				(path "/f756acf8-4d17-4038-8897-d8e944818549"
-					(reference "U3")
-					(unit 1)
-				)
-			)
-		)
-	)
-	(symbol
 		(lib_id "RF_Module:ESP32-S3-WROOM-1")
 		(at 190.5 80.01 0)
@@
 			)
 		)
-		(property "Footprint" "Capacitor_SMD:C_0603_1608Metric"
+		(property "Footprint" "Capacitor_SMD:C_0805_2012Metric"
 			(at 210.5152 45.72 0)
 			(effects
@@
 			)
 		)
-		(property "LCSC" "C59461"
+		(property "LCSC" "C45783"
 			(at 209.55 41.91 0)
 			(effects
@@
 			)
 		)
-		(property "Value" "0.1uF"
+		(property "Value" "10uF"
 			(at 108.966 44.45 0)
 			(effects
@@
 			)
 		)
-		(property "Footprint" "Capacitor_SMD:C_0603_1608Metric"
+		(property "Footprint" "Capacitor_SMD:C_0805_2012Metric"
 			(at 110.7948 46.99 0)
 			(effects
@@
 			)
 		)
-		(property "LCSC" "C14663"
+		(property "LCSC" "C15850"
 			(at 111.76 43.18 0)
 			(effects
@@
 	)
 	(symbol
-		(lib_id "Regulator_Linear:LD1117S33TR_SOT223")
+		(lib_id "ESP32_Dev_Board:AP2114H-3.3")
 		(at 124.46 38.1 0)
 		(unit 1)
@@
 			)
 		)
-		(property "Value" "LD1117S33TR_SOT223"
+		(property "Value" "AP2114H-3.3"
 			(at 124.46 34.29 0)
 			(effects
@@
 		)
 		(property "Footprint" "Package_TO_SOT_SMD:SOT-223-3_TabPin2"
-			(at 124.46 33.02 0)
+			(at 120.65 52.578 0)
 			(effects
 				(font
@@
 			)
 		)
-		(property "Datasheet" "http://www.st.com/st-web-ui/static/active/en/resource/technical/document/datasheet/CD00000544.pdf"
-			(at 127 44.45 0)
+		(property "Datasheet" "https://www.diodes.com/assets/Datasheets/AP2114.pdf"
+			(at 125.222 47.498 0)
 			(effects
 				(font
@@
 			)
 		)
-		(property "Description" "800mA Fixed Low Drop Positive Voltage Regulator, Fixed Output 3.3V, SOT-223"
-			(at 124.46 38.1 0)
+		(property "Description" "LDO Regulator, 1A, Fixed 3.3V, 2.5V-6V Input, Low Dropout, SOT-223"
+			(at 131.318 50.292 0)
 			(effects
 				(font
@@
 			)
 		)
-		(property "LCSC" "C86781"
+		(property "LCSC" "C150716"
 			(at 124.46 38.1 0)
 			(effects
@@
 			)
 		)
-		(property "LCSC" " C15849"
+		(property "LCSC" "C15849"
 			(at 162.56 62.23 0)
 			(effects
@@
 			)
 		)
-		(property "Value" "10uF"
+		(property "Value" "22uF"
 			(at 139.954 44.45 0)
 			(effects
@@
 			)
 		)
-		(property "Footprint" "Capacitor_SMD:C_0603_1608Metric"
+		(property "Footprint" "Capacitor_SMD:C_0805_2012Metric"
 			(at 138.1252 46.99 0)
 			(effects
@@
 			)
 		)
-		(property "LCSC" "C19702"
+		(property "LCSC" "C45783"
 			(at 137.16 43.18 0)
 			(effects
